File: scheme/main/control_isol.kicad_sch (KiCad schematic)
At the start: 33 parts, among them U14 CA-IS3760LW

Commit message: separate hi power & signal gnd
Connections:
- net GNDD renamed GND
- net GNDPWR renamed GNDH
