File: scheme/main/control_isol.kicad_sch (KiCad schematic)
At the start: 33 parts, among them U14 CA-IS3760LW

Commit message: sheets titles
Other:
- title: (none) -> Управление транзисторами
Changed lines of the file:
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@@
 	(generator_version "8.0")
 	(paper "A4")
+	(title_block
+		(title "Управление транзисторами")
+	)
 	(junction
 		(at 245.11 30.48)
