File: scheme/main/digital_output_single.kicad_sch (KiCad schematic)
At the start: 4 parts, among them K3 RM87N, Q3 BC847

Commit message: di & do terminals
Parts:
- renumbered D9 to D10, Q3 to Q4, R85 to R86
Changed lines of the file:
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@@
 		(on_board yes)
 		(dnp no)
-		(property "Reference" "D9"
+		(property "Reference" "D10"
 			(at 116.078 83.058 90)
 			(effects
@@
 		(dnp no)
 		(fields_autoplaced yes)
-		(property "Reference" "#PWR0104"
+		(property "Reference" "#PWR0106"
 			(at 142.24 115.57 0)
 			(effects
@@
 					(unit 1)
 				)
+				(path "/c11d1dbc-4db9-4712-8d1d-5f6f7086cded/7d40f93b-18df-4406-a354-a8dac5c853e3/97aa0c6a-3040-4632-b51b-83025e12675d"
+					(reference "K?")
+					(unit 1)
+				)
 			)
 		)
@@
 		(on_board yes)
 		(dnp no)
-		(property "Reference" "R85"
+		(property "Reference" "R86"
 			(at 122.682 107.188 90)
 			(effects
@@
 		(dnp no)
 		(fields_autoplaced yes)
-		(property "Reference" "#PWR0103"
+		(property "Reference" "#PWR0105"
 			(at 142.24 73.66 0)
 			(effects
@@
 		(dnp no)
 		(fields_autoplaced yes)
-		(property "Reference" "Q3"
+		(property "Reference" "Q4"
 			(at 144.78 100.3299 0)
 			(effects
