File: scheme/main/digital_output_single.kicad_sch (KiCad schematic)
At the start: 4 parts, among them K3 RM87N, Q4 BC847

Commit message: sheets titles
Other:
- title: (none) -> Цифровой выход
Changed lines of the file:
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@@
 	(generator_version "8.0")
 	(paper "A4")
+	(title_block
+		(title "Цифровой выход")
+	)
 	(junction
 		(at 127 76.2)
