File: scheme/main/digital_outputs.kicad_sch (KiCad schematic)
At the start: 0 parts

Commit message: sheets titles
Other:
- title: (none) -> Цифровые выходы
Changed lines of the file:
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@@
 	(generator_version "8.0")
 	(paper "A4")
+	(title_block
+		(title "Цифровые выходы")
+	)
 	(wire
 		(pts
