File: scheme/main/bus_term.kicad_sch (KiCad schematic)
At the start: 1 part, among them J2 Conn_01x03

Commit message: sheets titles
Other:
- title: (none) -> Клеммник цифровых шин
Changed lines of the file:
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@@
 	(generator_version "8.0")
 	(paper "A4")
+	(title_block
+		(title "Клеммник цифровых шин")
+	)
 	(wire
 		(pts

Commit message: footprints set/changed
Parts:
- J2: footprint (none) -> main:DG350-3.5-03P
Changed lines of the file:
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@@
 			)
 		)
-		(property "Footprint" ""
+		(property "Footprint" "main:DG350-3.5-03P"
 			(at 163.83 93.98 0)
 			(effects
