File: scheme/main/current_sense.kicad_sch (KiCad schematic)
At the start: 4 parts, among them U2 ACS712xLCTR-05B

Commit message: replace some 220n capacitors with 100n
Parts:
- C33: value 220nF -> 100nF
Changed lines of the file:
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@@
 			)
 		)
-		(property "Value" "220nF"
+		(property "Value" "100nF"
 			(at 135.89 102.8699 0)
 			(effects

Commit message: sheets titles
Other:
- title: (none) -> Датчик тока
Changed lines of the file:
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@@
 	(generator_version "8.0")
 	(paper "A4")
+	(title_block
+		(title "Датчик тока")
+	)
 	(junction
 		(at 119.38 111.76)

Commit message: removed current sensor out 22r resistors
Parts:
- removed R7: 22R, Resistor_SMD:R_0805_2012Metric, symbol Device:R
Connections:
- net OUT: now also U2.7 (VIOUT)
Changed lines of the file:
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@@
 	(wire
 		(pts
-			(xy 116.84 91.44) (xy 138.43 91.44)
-		)
-		(stroke
-			(width 0)
-			(type default)
-		)
-	)
-	(wire
-		(pts
-			(xy 146.05 91.44) (xy 151.13 91.44)
+			(xy 116.84 91.44) (xy 151.13 91.44)
 		)
 		(stroke
@@
 		)
 	)
-	(symbol
-		(lib_id "Device:R")
-		(at 142.24 91.44 90)
-		(unit 1)
-		(exclude_from_sim no)
-		(in_bom yes)
-		(on_board yes)
-		(dnp no)
-		(fields_autoplaced yes)
-		(property "Reference" "R7"
-			(at 142.24 85.09 90)
-			(effects
-				(font
-					(size 1.27 1.27)
-				)
-			)
-		)
-		(property "Value" "22R"
-			(at 142.24 87.63 90)
-			(effects
-				(font
-					(size 1.27 1.27)
-				)
-			)
-		)
-		(property "Footprint" "Resistor_SMD:R_0805_2012Metric"
-			(at 142.24 93.218 90)
-			(effects
-				(font
-					(size 1.27 1.27)
-				)
-				(hide yes)
-			)
-		)
-		(property "Datasheet" "~"
-			(at 142.24 91.44 0)
-			(effects
-				(font
-					(size 1.27 1.27)
-				)
-				(hide yes)
-			)
-		)
-		(property "Description" "Resistor"
-			(at 142.24 91.44 0)
-			(effects
-				(font
-					(size 1.27 1.27)
-				)
-				(hide yes)
-			)
-		)
-		(pin "1"
-		)
-		(pin "2"
-		)
-		(instances
-			(project "main"
-				(path "/c11d1dbc-4db9-4712-8d1d-5f6f7086cded/1bd0e084-5602-43f5-a9de-9167dc3ddabf"
-					(reference "R7")
-					(unit 1)
-				)
-				(path "/c11d1dbc-4db9-4712-8d1d-5f6f7086cded/236c27c1-9285-48af-b94c-0a581f89ad4f"
-					(reference "R145")
-					(unit 1)
-				)
-				(path "/c11d1dbc-4db9-4712-8d1d-5f6f7086cded/eb061644-a076-485c-afde-65b59d5b34e4"
-					(reference "R8")
-					(unit 1)
-				)
-			)
-		)
-	)
