File: scheme/main/digital_input_single.kicad_sch (KiCad schematic)
At the start: 7 parts, among them U23 PC817

Commit message: added input buffer
Parts:
- removed R110: 22R, Resistor_SMD:R_0805_2012Metric, symbol Device:R
Connections:
- net out: now also R79.2, U23.3
Changed lines of the file:
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@@
 	(wire
 		(pts
-			(xy 190.5 95.25) (xy 193.04 95.25)
+			(xy 190.5 95.25) (xy 203.2 95.25)
 		)
 		(stroke
@@
 		(pts
 			(xy 149.86 95.25) (xy 137.16 95.25)
-		)
-		(stroke
-			(width 0)
-			(type default)
-		)
-	)
-	(wire
-		(pts
-			(xy 200.66 95.25) (xy 203.2 95.25)
 		)
 		(stroke
@@
 					(unit 1)
 				)
-			)
-		)
-	)
-	(symbol
-		(lib_id "Device:R")
-		(at 196.85 95.25 90)
-		(unit 1)
-		(exclude_from_sim no)
-		(in_bom yes)
-		(on_board yes)
-		(dnp no)
-		(fields_autoplaced yes)
-		(property "Reference" "R110"
-			(at 196.85 88.9 90)
-			(effects
-				(font
-					(size 1.27 1.27)
-				)
-			)
-		)
-		(property "Value" "22R"
-			(at 196.85 91.44 90)
-			(effects
-				(font
-					(size 1.27 1.27)
-				)
-			)
-		)
-		(property "Footprint" "Resistor_SMD:R_0805_2012Metric"
-			(at 196.85 97.028 90)
-			(effects
-				(font
-					(size 1.27 1.27)
-				)
-				(hide yes)
-			)
-		)
-		(property "Datasheet" "~"
-			(at 196.85 95.25 0)
-			(effects
-				(font
-					(size 1.27 1.27)
-				)
-				(hide yes)
-			)
-		)
-		(property "Description" "Resistor"
-			(at 196.85 95.25 0)
-			(effects
-				(font
-					(size 1.27 1.27)
-				)
-				(hide yes)
-			)
-		)
-		(pin "1"
-		)
-		(pin "2"
-		)
-		(instances
-			(project "main"
-				(path "/c11d1dbc-4db9-4712-8d1d-5f6f7086cded/bedea6de-a196-4917-ba70-c071156ad9b9/31162724-615b-46ba-8c0e-f604e9ec35b9"
-					(reference "R110")
-					(unit 1)
-				)
-				(path "/c11d1dbc-4db9-4712-8d1d-5f6f7086cded/bedea6de-a196-4917-ba70-c071156ad9b9/9dc33930-f682-4ed1-a57d-b39bd6b7930d"
-					(reference "R109")
-					(unit 1)
-				)
-				(path "/c11d1dbc-4db9-4712-8d1d-5f6f7086cded/bedea6de-a196-4917-ba70-c071156ad9b9/a9420b45-d901-4429-a945-3bcdca919a43"
-					(reference "R108")
-					(unit 1)
-				)
-				(path "/c11d1dbc-4db9-4712-8d1d-5f6f7086cded/bedea6de-a196-4917-ba70-c071156ad9b9/bd001503-3ad8-4979-953f-3e7ea894eb19"
-					(reference "R111")
-					(unit 1)
-				)

Commit message: sheets titles
Other:
- title: (none) -> Цифровой вход
Changed lines of the file:
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@@
 	(generator_version "8.0")
 	(paper "A4")
+	(title_block
+		(title "Цифровой вход")
+	)
 	(junction
 		(at 125.73 82.55)
