File: scheme/main/digital_output_term.kicad_sch (KiCad schematic)
At the start: 1 part, among them X2 DG142V-06P_5.08

Commit message: added 24V & GND to DO terminal & more
Parts:
- removed X2: DG142V-06P_5.08, main:DG142V-06P-5.08_V1.0, symbol main:DG142V-06P_5.08
- added X2: DG142V-08P_5.08, main:DG142V-08P-5.08_V1.0, symbol main:DG142V-08P_5.08
Connections:
- net DO1_COM: now also X2.4
- net DO1_NC: now also X2.2
- net DO1_NO: now also X2.3
- net DO2_COM: now also X2.7
- net DO2_NC: now also X2.5
- net DO2_NO: now also X2.6
- new net +24V: X2.1
- new net GND: X2.8
Changed lines of the file:
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@@
+	(wire
+		(pts
+			(xy 157.48 77.47) (xy 157.48 74.93)
+		)
+		(stroke
+			(width 0)
+			(type default)
+		)
+	)
+	(wire
+		(pts
+			(xy 160.02 77.47) (xy 157.48 77.47)
+		)
+		(stroke
+			(width 0)
+			(type default)
+		)
+	)
 	(wire
 		(pts
@@
 	(wire
 		(pts
+			(xy 157.48 95.25) (xy 157.48 97.79)
+		)
+		(stroke
+			(width 0)
+			(type default)
+		)
+	)
+	(wire
+		(pts
+			(xy 160.02 95.25) (xy 157.48 95.25)
+		)
+		(stroke
+			(width 0)
+			(type default)
+		)
+	)
+	(wire
+		(pts
 			(xy 149.86 82.55) (xy 160.02 82.55)
 		)
@@
 	)
 	(symbol
-		(lib_id "main:DG142V-06P_5.08")
-		(at 165.1 78.74 0)
+		(lib_id "power:GND")
+		(at 157.48 97.79 0)
+		(unit 1)
+		(exclude_from_sim no)
+		(in_bom yes)
+		(on_board yes)
+		(dnp no)
+		(fields_autoplaced yes)
+		(property "Reference" "#PWR151"
+			(at 157.48 104.14 0)
+			(effects
+				(font
+					(size 1.27 1.27)
+				)
+				(hide yes)
+			)
+		)
+		(property "Value" "GND"
+			(at 157.48 102.87 0)
+			(effects
+				(font
+					(size 1.27 1.27)
+				)
+			)
+		)
+		(property "Footprint" ""
+			(at 157.48 97.79 0)
+			(effects
+				(font
+					(size 1.27 1.27)
+				)
+				(hide yes)
+			)
+		)
+		(property "Datasheet" ""
+			(at 157.48 97.79 0)
+			(effects
+				(font
+					(size 1.27 1.27)
+				)
+				(hide yes)
+			)
+		)
+		(property "Description" "Power symbol creates a global label with name \"GND\" , ground"
+			(at 157.48 97.79 0)
+			(effects
+				(font
+					(size 1.27 1.27)
+				)
+				(hide yes)
+			)
+		)
+		(pin "1"
+		)
+		(instances
+			(project "main"
+				(path "/c11d1dbc-4db9-4712-8d1d-5f6f7086cded/5fa6ede8-f1b3-46e0-b9d4-c21c084d88c4"
+					(reference "#PWR151")
+					(unit 1)
+				)
+			)
+		)
+	)
+	(symbol
+		(lib_id "power:+24V")
+		(at 157.48 74.93 0)
+		(unit 1)
+		(exclude_from_sim no)
+		(in_bom yes)
+		(on_board yes)
+		(dnp no)
+		(fields_autoplaced yes)
+		(property "Reference" "#PWR150"
+			(at 157.48 78.74 0)
+			(effects
+				(font
+					(size 1.27 1.27)
+				)
+				(hide yes)
+			)
+		)
+		(property "Value" "+24V"
+			(at 157.48 69.85 0)
+			(effects
+				(font
+					(size 1.27 1.27)
+				)
+			)
+		)
+		(property "Footprint" ""
+			(at 157.48 74.93 0)
+			(effects
+				(font
+					(size 1.27 1.27)
+				)
+				(hide yes)
+			)
+		)
+		(property "Datasheet" ""
+			(at 157.48 74.93 0)
+			(effects
+				(font
+					(size 1.27 1.27)
+				)
+				(hide yes)
+			)
+		)
+		(property "Description" "Power symbol creates a global label with name \"+24V\""
+			(at 157.48 74.93 0)
+			(effects
+				(font
+					(size 1.27 1.27)
+				)
+				(hide yes)
+			)
+		)
+		(pin "1"
+		)
+		(instances
+			(project "main"
+				(path "/c11d1dbc-4db9-4712-8d1d-5f6f7086cded/5fa6ede8-f1b3-46e0-b9d4-c21c084d88c4"
+					(reference "#PWR150")
+					(unit 1)
+				)
+			)
+		)
+	)
+	(symbol
+		(lib_id "main:DG142V-08P_5.08")
+		(at 165.1 76.2 0)
 		(mirror y)
 		(unit 1)
@@
 			)
 		)
-		(property "Value" "DG142V-06P_5.08"
+		(property "Value" "DG142V-08P_5.08"
 			(at 166.37 87.6299 0)
 			(effects
@@
 			)
 		)
-		(property "Footprint" "main:DG142V-06P-5.08_V1.0"
-			(at 156.718 99.06 0)
-			(effects
-				(font
-					(size 1.27 1.27)
-				)
-				(hide yes)
-			)
-		)
-		(property "Datasheet" "https://www.platan.ru/cgi-bin/qwery.pl/id=2010019306"
-			(at 155.702 102.616 0)
+		(property "Footprint" "main:DG142V-08P-5.08_V1.0"
+			(at 156.718 96.52 0)
+			(effects
+				(font
+					(size 1.27 1.27)
+				)
+				(hide yes)
+			)
+		)
+		(property "Datasheet" ""
+			(at 155.702 100.076 0)
 			(effects
 				(font
@@
 		)
 		(property "Description" ""
-			(at 165.1 78.74 0)
-			(effects
-				(font
-					(size 1.27 1.27)
-				)
-				(hide yes)
-			)
-		)
-		(property "Manufacturer Part" "DG142V-5.08-06P"
-			(at 155.956 95.758 0)
-			(effects
-				(font
-					(size 1.27 1.27)
-				)
-				(hide yes)
-			)
+			(at 165.1 76.2 0)
+			(effects
+				(font
+					(size 1.27 1.27)
+				)
+				(hide yes)
+			)
+		)
+		(property "Manufacturer Part" "DG142V-5.08-08P"
+			(at 175.768 87.884 0)
+			(effects
+				(font
+					(size 1.27 1.27)
+				)
+				(hide yes)
+			)
+		)
+		(pin "3"
+		)
+		(pin "7"
+		)
+		(pin "2"
+		)
+		(pin "5"
+		)
+		(pin "6"
+		)
+		(pin "1"
 		)
 		(pin "4"
 		)
-		(pin "2"
-		)
-		(pin "5"
-		)
-		(pin "1"
-		)
-		(pin "6"
-		)
-		(pin "3"
+		(pin "8"
 		)
 		(instances

Commit message: sheets titles
Other:
- title: (none) -> Клеммник цифровых выходов
Changed lines of the file:
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@@
 	(generator_version "8.0")
 	(paper "A4")
+	(title_block
+		(title "Клеммник цифровых выходов")
+	)
 	(wire
 		(pts
