File: scheme/main/input_buffer.kicad_sch (KiCad schematic)
At the start: 8 parts, among them U27 74HC244

Commit message: added 24V & GND to DO terminal & more
Changed lines of the file:
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@@
 	(paper "A4")
 	(junction
+		(at 153.67 97.79)
+		(diameter 0)
+		(color 0 0 0 0)
+	)
+	(junction
 		(at 153.67 63.5)
 		(diameter 0)
@@
 	)
 	(junction
-		(at 162.56 88.9)
+		(at 162.56 97.79)
 		(diameter 0)
 		(color 0 0 0 0)
@@
 	)
 	(junction
-		(at 153.67 88.9)
-		(diameter 0)
-		(color 0 0 0 0)
-	)
-	(junction
-		(at 171.45 88.9)
-		(diameter 0)
-		(color 0 0 0 0)
-	)
-	(junction
-		(at 180.34 88.9)
+		(at 171.45 97.79)
+		(diameter 0)
+		(color 0 0 0 0)
+	)
+	(junction
+		(at 180.34 97.79)
 		(diameter 0)
 		(color 0 0 0 0)
@@
 	(wire
 		(pts
-			(xy 162.56 86.36) (xy 162.56 88.9)
+			(xy 162.56 86.36) (xy 162.56 97.79)
 		)
 		(stroke
@@
 	(wire
 		(pts
-			(xy 180.34 86.36) (xy 180.34 88.9)
-		)
-		(stroke
-			(width 0)
-			(type default)
-		)
-	)
-	(wire
-		(pts
-			(xy 162.56 88.9) (xy 171.45 88.9)
+			(xy 180.34 86.36) (xy 180.34 97.79)
+		)
+		(stroke
+			(width 0)
+			(type default)
+		)
+	)
+	(wire
+		(pts
+			(xy 162.56 97.79) (xy 171.45 97.79)
 		)
 		(stroke
@@
 	(wire
 		(pts
-			(xy 180.34 88.9) (xy 189.23 88.9)
+			(xy 180.34 97.79) (xy 189.23 97.79)
 		)
 		(stroke
@@
 	(wire
 		(pts
-			(xy 153.67 88.9) (xy 162.56 88.9)
+			(xy 153.67 97.79) (xy 162.56 97.79)
 		)
 		(stroke
@@
 	(wire
 		(pts
-			(xy 153.67 86.36) (xy 153.67 88.9)
-		)
-		(stroke
-			(width 0)
-			(type default)
-		)
-	)
-	(wire
-		(pts
 			(xy 143.51 68.58) (xy 171.45 68.58)
 		)
@@
 	(wire
 		(pts
-			(xy 153.67 97.79) (xy 153.67 88.9)
-		)
-		(stroke
-			(width 0)
-			(type default)
-		)
-	)
-	(wire
-		(pts
-			(xy 189.23 86.36) (xy 189.23 88.9)
+			(xy 153.67 86.36) (xy 153.67 97.79)
+		)
+		(stroke
+			(width 0)
+			(type default)
+		)
+	)
+	(wire
+		(pts
+			(xy 189.23 86.36) (xy 189.23 97.79)
 		)
 		(stroke
@@
 	(wire
 		(pts
-			(xy 171.45 88.9) (xy 180.34 88.9)
+			(xy 171.45 97.79) (xy 180.34 97.79)
 		)
 		(stroke
@@
 	(wire
 		(pts
-			(xy 171.45 86.36) (xy 171.45 88.9)
-		)
-		(stroke
+			(xy 171.45 86.36) (xy 171.45 97.79)
+		)
+		(stroke

Commit message: sheets titles
Other:
- title: (none) -> Входные буферы
Changed lines of the file:
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@@
 	(generator_version "8.0")
 	(paper "A4")
+	(title_block
+		(title "Входные буферы")
+	)
 	(junction
 		(at 153.67 97.79)

Commit message: footprints set/changed
Parts:
- U27: footprint (none) -> Package_SO:SOIC-20W_7.5x12.8mm_P1.27mm
Changed lines of the file:
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@@
 			)
 		)
-		(property "Footprint" ""
+		(property "Footprint" "Package_SO:SOIC-20W_7.5x12.8mm_P1.27mm"
 			(at 130.81 76.2 0)
 			(effects
