File: scheme/main/itrip.kicad_sch (KiCad schematic)
At the start: 16 parts

Commit message: added L fuse & more
Parts:
- NT2: footprint (none) -> NetTie:NetTie-2_SMD_Pad0.5mm
Changed lines of the file:
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@@
 			)
 		)
-		(property "Footprint" ""
+		(property "Footprint" "NetTie:NetTie-2_SMD_Pad0.5mm"
 			(at 156.21 129.54 0)
 			(effects

Commit message: sheets titles
Other:
- title: (none) -> Токовая защита
Changed lines of the file:
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@@
 	(generator_version "8.0")
 	(paper "A4")
+	(title_block
+		(title "Токовая защита")
+	)
 	(junction
 		(at 113.03 113.03)
