File: scheme/main/main.kicad_sch (KiCad schematic)
At the start: 0 parts

Commit message: sheets titles
Other:
- title: (none) -> Частотный преобразователь
Changed lines of the file:
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@@
 	(generator_version "8.0")
 	(paper "A4")
+	(title_block
+		(title "Частотный преобразователь")
+	)
 	(junction
 		(at 53.34 147.32)

Commit message: added analog input 0 && sheets sort
Other:
- added sheet analog_input (analog_input.kicad_sch)
- added sheet analog_input_term (analog_input_term.kicad_sch)
- sheet ctrl_con ports: added ain0; removed none
Changed lines of the file:
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@@
+	(wire
+		(pts
+			(xy 77.47 173.99) (xy 101.6 173.99)
+		)
+		(stroke
+			(width 0)
+			(type default)
+		)
+	)
 	(wire
 		(pts
@@
 	(wire
 		(pts
-			(xy 90.17 133.35) (xy 90.17 107.95)
+			(xy 90.17 133.35) (xy 90.17 110.49)
 		)
 		(stroke
@@
 	(wire
 		(pts
-			(xy 92.71 110.49) (xy 116.84 110.49)
+			(xy 92.71 113.03) (xy 116.84 113.03)
 		)
 		(stroke
@@
 	(wire
 		(pts
-			(xy 92.71 139.7) (xy 92.71 110.49)
+			(xy 92.71 139.7) (xy 92.71 113.03)
 		)
 		(stroke
@@
 	(wire
 		(pts
+			(xy 101.6 173.99) (xy 101.6 102.87)
+		)
+		(stroke
+			(width 0)
+			(type default)
+		)
+	)
+	(wire
+		(pts
+			(xy 101.6 102.87) (xy 116.84 102.87)
+		)
+		(stroke
+			(width 0)
+			(type default)
+		)
+	)
+	(wire
+		(pts
 			(xy 60.96 30.48) (xy 72.39 30.48)
 		)
@@
 	(wire
 		(pts
+			(xy 40.64 173.99) (xy 57.15 173.99)
+		)
+		(stroke
+			(width 0)
+			(type default)
+		)
+	)
+	(wire
+		(pts
 			(xy 170.18 40.64) (xy 170.18 19.05)
 		)
@@
 	(wire
 		(pts
-			(xy 95.25 146.05) (xy 95.25 113.03)
+			(xy 95.25 146.05) (xy 95.25 115.57)
 		)
 		(stroke
@@
 	(wire
 		(pts
-			(xy 95.25 113.03) (xy 116.84 113.03)
+			(xy 95.25 115.57) (xy 116.84 115.57)
 		)
 		(stroke
@@
 	(wire
 		(pts
-			(xy 90.17 107.95) (xy 116.84 107.95)
+			(xy 90.17 110.49) (xy 116.84 110.49)
 		)
 		(stroke
@@
 	(wire
 		(pts
-			(xy 106.68 104.14) (xy 116.84 104.14)
+			(xy 106.68 106.68) (xy 116.84 106.68)
 		)
 		(stroke
@@
 	(wire
 		(pts
-			(xy 106.68 129.54) (xy 106.68 104.14)
+			(xy 106.68 129.54) (xy 106.68 106.68)
 		)
 		(stroke
@@
 	(wire
 		(pts
-			(xy 97.79 115.57) (xy 116.84 115.57)
+			(xy 97.79 118.11) (xy 116.84 118.11)
 		)
 		(stroke
@@
 	(wire
 		(pts
-			(xy 97.79 152.4) (xy 97.79 115.57)
+			(xy 97.79 152.4) (xy 97.79 118.11)
 		)
 		(stroke
@@
 			(project "main"
 				(path "/c11d1dbc-4db9-4712-8d1d-5f6f7086cded"
-					(page "4")
+					(page "24")
 				)
 			)
@@
 			(project "main"
 				(path "/c11d1dbc-4db9-4712-8d1d-5f6f7086cded"
-					(page "2")
+					(page "22")
 				)
 			)
@@
 			(project "main"
 				(path "/c11d1dbc-4db9-4712-8d1d-5f6f7086cded"
-					(page "3")
+					(page "23")
 				)
 			)
@@
 			(project "main"
 				(path "/c11d1dbc-4db9-4712-8d1d-5f6f7086cded"
-					(page "28")
+					(page "39")
 				)
 			)
@@
 			(project "main"
 				(path "/c11d1dbc-4db9-4712-8d1d-5f6f7086cded"
-					(page "17")
+					(page "30")
 				)
 			)
@@
 			(project "main"
 				(path "/c11d1dbc-4db9-4712-8d1d-5f6f7086cded"
-					(page "7")
+					(page "27")
 				)
 			)
@@
 	(sheet
 		(at 160.02 85.09)
-		(size 27.94 34.29)
+		(size 27.94 35.56)
 		(fields_autoplaced yes)
 		(stroke
@@
 		)
 		(property "Sheetfile" "ipm.kicad_sch"
-			(at 160.02 119.9646 0)
+			(at 160.02 121.2346 0)
 			(effects
 				(font
@@
 			(project "main"
 				(path "/c11d1dbc-4db9-4712-8d1d-5f6f7086cded"
-					(page "8")
+					(page "2")
 				)
 			)
@@
 			(project "main"
 				(path "/c11d1dbc-4db9-4712-8d1d-5f6f7086cded"
-					(page "27")
+					(page "43")
 				)
 			)
@@
 			(project "main"
 				(path "/c11d1dbc-4db9-4712-8d1d-5f6f7086cded"
-					(page "15")
+					(page "28")
 				)
 			)
@@
 			(project "main"
 				(path "/c11d1dbc-4db9-4712-8d1d-5f6f7086cded"
-					(page "24")
+					(page "40")
 				)
 			)
@@
 			(project "main"
 				(path "/c11d1dbc-4db9-4712-8d1d-5f6f7086cded"
-					(page "18")
+					(page "31")
 				)
 			)
@@
 			(project "main"
 				(path "/c11d1dbc-4db9-4712-8d1d-5f6f7086cded"
-					(page "5")
+					(page "25")
 				)
 			)
@@
 			(project "main"
 				(path "/c11d1dbc-4db9-4712-8d1d-5f6f7086cded"
-					(page "19")
+					(page "34")
+				)
+			)
+		)
+	)
+	(sheet
+		(at 57.15 171.45)
+		(size 20.32 5.08)
+		(fields_autoplaced yes)
+		(stroke
+			(width 0.1524)
+			(type solid)
+		)
+		(fill
+			(color 0 0 0 0.0000)
+		)
+		(property "Sheetname" "analog_input"
+			(at 57.15 170.7384 0)
+			(effects
+				(font
+					(size 1.27 1.27)
+				)
+				(justify left bottom)
+			)
+		)
+		(property "Sheetfile" "analog_input.kicad_sch"
+			(at 57.15 177.1146 0)
+			(effects
+				(font
+					(size 1.27 1.27)
+				)
+				(justify left top)
+			)
+		)
+		(pin "AIN0_IN" input
+			(at 57.15 173.99 180)
+			(effects
+				(font
+					(size 1.27 1.27)
+				)
+				(justify left)
+			)
+		)
+		(pin "AIN0_OUT" output
+			(at 77.47 173.99 0)
+			(effects
+				(font
+					(size 1.27 1.27)
+				)
+				(justify right)
+			)
+		)
+		(instances
+			(project "main"
+				(path "/c11d1dbc-4db9-4712-8d1d-5f6f7086cded"
+					(page "44")
+				)
+			)
+		)
+	)
+	(sheet
+		(at 20.32 171.45)
+		(size 20.32 5.08)
+		(fields_autoplaced yes)
+		(stroke
+			(width 0.1524)
+			(type solid)
+		)
+		(fill
+			(color 0 0 0 0.0000)
+		)
+		(property "Sheetname" "analog_input_term"
+			(at 20.32 170.7384 0)
+			(effects
+				(font
+					(size 1.27 1.27)
+				)
+				(justify left bottom)
+			)
+		)
+		(property "Sheetfile" "analog_input_term.kicad_sch"
+			(at 20.32 177.1146 0)
+			(effects
+				(font
+					(size 1.27 1.27)
+				)
+				(justify left top)
+			)
+		)
+		(pin "AIN0" output
+			(at 40.64 173.99 0)
+			(effects
+				(font
+					(size 1.27 1.27)
+				)
+				(justify right)
+			)
+		)
+		(instances
+			(project "main"
+				(path "/c11d1dbc-4db9-4712-8d1d-5f6f7086cded"
+					(page "46")
 				)
 			)
@@
 			(project "main"
 				(path "/c11d1dbc-4db9-4712-8d1d-5f6f7086cded"
-					(page "30")
+					(page "32")
 				)
 			)
@@
 	(sheet
 		(at 116.84 85.09)
-		(size 27.94 34.29)
+		(size 27.94 35.56)
 		(fields_autoplaced yes)
 		(stroke
@@
 		)
 		(property "Sheetfile" "ctrl_con.kicad_sch"
-			(at 116.84 119.9646 0)
+			(at 116.84 121.2346 0)
 			(effects
 				(font
@@
 		)
 		(pin "Trip" input
-			(at 116.84 104.14 180)
+			(at 116.84 106.68 180)
 			(effects
 				(font
@@
 		)
 		(pin "di1" input
-			(at 116.84 107.95 180)
+			(at 116.84 110.49 180)
 			(effects
 				(font
@@
 		)
 		(pin "di2" input
-			(at 116.84 110.49 180)
+			(at 116.84 113.03 180)
 			(effects
 				(font
@@
 		)
 		(pin "di3" input
-			(at 116.84 113.03 180)
+			(at 116.84 115.57 180)
 			(effects
 				(font
@@
 		)
 		(pin "di4" input
-			(at 116.84 115.57 180)
+			(at 116.84 118.11 180)
 			(effects
 				(font
@@
 				)
 				(justify right)
+			)
+		)
+		(pin "ain0" input
+			(at 116.84 102.87 180)
+			(effects
+				(font
+					(size 1.27 1.27)
+				)
+				(justify left)
 			)
 		)
@@
 			(project "main"
 				(path "/c11d1dbc-4db9-4712-8d1d-5f6f7086cded"
-					(page "31")
+					(page "10")
 				)
 			)
@@
 			(project "main"
 				(path "/c11d1dbc-4db9-4712-8d1d-5f6f7086cded"
-					(page "6")
+					(page "26")
 				)
 			)
@@
 			(project "main"
 				(path "/c11d1dbc-4db9-4712-8d1d-5f6f7086cded"
-					(page "16")
+					(page "29")
 				)
 			)
@@
 			(project "main"
 				(path "/c11d1dbc-4db9-4712-8d1d-5f6f7086cded"
-					(page "29")
-				)
-			)
+					(page "33")
+				)
+			)
