File: scheme/main/output_buffer.kicad_sch (KiCad schematic)
At the start: 15 parts, among them U25 74HC244, U26 74HC244

Commit message: added 24V & GND to DO terminal & more
Changed lines of the file:
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@@
-	)
-	(junction
-		(at 137.16 160.02)
-		(diameter 0)
-		(color 0 0 0 0)
 	)
 	(junction
@@
 	)
 	(junction
-		(at 154.94 74.93)
+		(at 154.94 83.82)
 		(diameter 0)
 		(color 0 0 0 0)
@@
 	)
 	(junction
-		(at 172.72 74.93)
+		(at 172.72 83.82)
 		(diameter 0)
 		(color 0 0 0 0)
@@
 	)
 	(junction
-		(at 146.05 74.93)
+		(at 146.05 83.82)
 		(diameter 0)
 		(color 0 0 0 0)
@@
 	)
 	(junction
-		(at 137.16 74.93)
+		(at 137.16 168.91)
 		(diameter 0)
 		(color 0 0 0 0)
@@
 	)
 	(junction
-		(at 146.05 160.02)
+		(at 146.05 168.91)
 		(diameter 0)
 		(color 0 0 0 0)
@@
 	)
 	(junction
-		(at 163.83 74.93)
+		(at 163.83 83.82)
 		(diameter 0)
 		(color 0 0 0 0)
@@
 	(junction
 		(at 99.06 72.39)
+		(diameter 0)
+		(color 0 0 0 0)
+	)
+	(junction
+		(at 137.16 83.82)
 		(diameter 0)
 		(color 0 0 0 0)
@@
 	(wire
 		(pts
+			(xy 154.94 72.39) (xy 154.94 83.82)
+		)
+		(stroke
+			(width 0)
+			(type default)
+		)
+	)
+	(wire
+		(pts
 			(xy 172.72 59.69) (xy 189.23 59.69)
 		)
@@
 	(wire
 		(pts
-			(xy 137.16 160.02) (xy 146.05 160.02)
+			(xy 137.16 168.91) (xy 146.05 168.91)
 		)
 		(stroke
@@
 	(wire
 		(pts
-			(xy 137.16 157.48) (xy 137.16 160.02)
+			(xy 137.16 72.39) (xy 137.16 83.82)
 		)
 		(stroke
@@
 	(wire
 		(pts
-			(xy 163.83 74.93) (xy 172.72 74.93)
+			(xy 163.83 83.82) (xy 172.72 83.82)
 		)
 		(stroke
@@
 	(wire
 		(pts
-			(xy 181.61 72.39) (xy 181.61 74.93)
-		)
-		(stroke
-			(width 0)
-			(type default)
-		)
-	)
-	(wire
-		(pts
 			(xy 101.6 72.39) (xy 99.06 72.39)
 		)
@@
 	(wire
 		(pts
+			(xy 137.16 157.48) (xy 137.16 168.91)
+		)
+		(stroke
+			(width 0)
+			(type default)
+		)
+	)
+	(wire
+		(pts
 			(xy 72.39 72.39) (xy 93.98 72.39)
 		)
@@
 	(wire
 		(pts
-			(xy 146.05 157.48) (xy 146.05 160.02)
+			(xy 146.05 157.48) (xy 146.05 168.91)
 		)
 		(stroke
@@
 	(wire
 		(pts
-			(xy 154.94 74.93) (xy 163.83 74.93)
+			(xy 154.94 83.82) (xy 163.83 83.82)
 		)
 		(stroke
@@
 	(wire
 		(pts
+			(xy 181.61 72.39) (xy 181.61 83.82)
+		)
+		(stroke
+			(width 0)
+			(type default)
+		)
+	)
+	(wire
+		(pts
 			(xy 137.16 134.62) (xy 137.16 149.86)
 		)
@@
 	(wire
 		(pts
-			(xy 137.16 168.91) (xy 137.16 160.02)
-		)
-		(stroke
-			(width 0)
-			(type default)
-		)
-	)
-	(wire
-		(pts
 			(xy 72.39 57.15) (xy 101.6 57.15)
 		)
@@
 	(wire
 		(pts
-			(xy 146.05 160.02) (xy 154.94 160.02)
+			(xy 146.05 168.91) (xy 154.94 168.91)
 		)
 		(stroke
@@
 	(wire
 		(pts
-			(xy 172.72 72.39) (xy 172.72 74.93)
-		)
-		(stroke
-			(width 0)
-			(type default)
-		)
-	)
-	(wire
-		(pts
-			(xy 154.94 72.39) (xy 154.94 74.93)
+			(xy 172.72 72.39) (xy 172.72 83.82)
 		)
 		(stroke
@@
 	(wire
 		(pts
-			(xy 137.16 72.39) (xy 137.16 74.93)
-		)
-		(stroke
-			(width 0)
-			(type default)
-		)
-	)
-	(wire
-		(pts
 			(xy 127 52.07) (xy 146.05 52.07)
 		)
@@
 	(wire
 		(pts
-			(xy 172.72 74.93) (xy 181.61 74.93)
+			(xy 172.72 83.82) (xy 181.61 83.82)
 		)
 		(stroke
@@
 	(wire
 		(pts
-			(xy 154.94 157.48) (xy 154.94 160.02)
+			(xy 154.94 157.48) (xy 154.94 168.91)
 		)
 		(stroke
@@
 	(wire
 		(pts
-			(xy 146.05 74.93) (xy 154.94 74.93)
+			(xy 146.05 83.82) (xy 154.94 83.82)
 		)
 		(stroke
@@
 	(wire
 		(pts
-			(xy 137.16 74.93) (xy 146.05 74.93)
+			(xy 137.16 83.82) (xy 146.05 83.82)
 		)
 		(stroke
@@
 	(wire
 		(pts
-			(xy 137.16 83.82) (xy 137.16 74.93)
-		)
-		(stroke
-			(width 0)
-			(type default)
-		)
-	)
-	(wire
-		(pts
 			(xy 99.06 147.32) (xy 101.6 147.32)
 		)
@@
 	(wire
 		(pts
-			(xy 146.05 72.39) (xy 146.05 74.93)
+			(xy 146.05 72.39) (xy 146.05 83.82)
 		)
 		(stroke
@@
 	(wire
 		(pts
-			(xy 163.83 72.39) (xy 163.83 74.93)
-		)
-		(stroke
+			(xy 163.83 72.39) (xy 163.83 83.82)
+		)
+		(stroke

Commit message: sheets titles
Other:
- title: (none) -> Выходные буферы
Changed lines of the file:
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@@
 	(generator_version "8.0")
 	(paper "A4")
+	(title_block
+		(title "Выходные буферы")
+	)
 	(junction
 		(at 146.05 52.07)

Commit message: added output buffers OE pull-down optional resistors
Parts:
- added R148, R149: 10k, Resistor_SMD:R_0805_2012Metric, symbol Device:R
Connections:
- net GND: now also R148.2, R149.2
- net oe: now also R149.1
- net pwm_oe: now also R148.1
Other:
- note added: "Паять один из двух резисторов-подтяжек OE."
Changed lines of the file:
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@@
+	)
+	(junction
+		(at 96.52 83.82)
+		(diameter 0)
+		(color 0 0 0 0)
 	)
 	(junction
@@
 	(junction
 		(at 114.3 36.83)
+		(diameter 0)
+		(color 0 0 0 0)
+	)
+	(junction
+		(at 96.52 168.91)
 		(diameter 0)
 		(color 0 0 0 0)
@@
 	(wire
 		(pts
+			(xy 93.98 82.55) (xy 93.98 83.82)
+		)
+		(stroke
+			(width 0)
+			(type default)
+		)
+	)
+	(wire
+		(pts
 			(xy 163.83 83.82) (xy 172.72 83.82)
 		)
@@
 	(wire
 		(pts
+			(xy 93.98 83.82) (xy 96.52 83.82)
+		)
+		(stroke
+			(width 0)
+			(type default)
+		)
+	)
+	(wire
+		(pts
 			(xy 137.16 157.48) (xy 137.16 168.91)
 		)
@@
 	(wire
 		(pts
+			(xy 93.98 72.39) (xy 93.98 74.93)
+		)
+		(stroke
+			(width 0)
+			(type default)
+		)
+	)
+	(wire
+		(pts
 			(xy 72.39 72.39) (xy 93.98 72.39)
 		)
@@
 	(wire
 		(pts
+			(xy 93.98 167.64) (xy 93.98 168.91)
+		)
+		(stroke
+			(width 0)
+			(type default)
+		)
+	)
+	(wire
+		(pts
 			(xy 99.06 72.39) (xy 99.06 74.93)
 		)
@@
 	(wire
 		(pts
+			(xy 93.98 157.48) (xy 93.98 160.02)
+		)
+		(stroke
+			(width 0)
+			(type default)
+		)
+	)
+	(wire
+		(pts
 			(xy 72.39 57.15) (xy 101.6 57.15)
 		)
@@
 			(width 0)
 			(type default)
+		)
+	)
+	(wire
+		(pts
+			(xy 93.98 168.91) (xy 96.52 168.91)
+		)
+		(stroke
+			(width 0)
+			(type default)
+		)
+	)
+	(text "Паять один из двух\nрезисторов-подтяжек OE."
+		(exclude_from_sim no)
+		(at 78.232 67.818 0)
+		(effects
+			(font
+				(size 1.27 1.27)
+			)
+		)
+	)
+	(text "Паять один из двух\nрезисторов-подтяжек OE."
+		(exclude_from_sim no)
+		(at 78.232 152.908 0)
+		(effects
+			(font
+				(size 1.27 1.27)
+			)
 		)
 	)
@@
 			)
 			(justify left)
+		)
+	)
+	(symbol
+		(lib_id "Device:R")
+		(at 93.98 78.74 0)
+		(mirror y)
+		(unit 1)
+		(exclude_from_sim no)
+		(in_bom yes)
+		(on_board yes)
+		(dnp yes)
+		(property "Reference" "R148"
+			(at 89.662 77.216 0)
+			(effects
+				(font
+					(size 1.27 1.27)
+				)
+			)
+		)
+		(property "Value" "10k"
+			(at 89.662 80.01 0)
+			(effects
+				(font
+					(size 1.27 1.27)
+				)
+			)
+		)
+		(property "Footprint" "Resistor_SMD:R_0805_2012Metric"
+			(at 95.758 78.74 90)
+			(effects
+				(font
+					(size 1.27 1.27)
+				)
+				(hide yes)
+			)
+		)
+		(property "Datasheet" "~"
+			(at 93.98 78.74 0)
+			(effects
+				(font
+					(size 1.27 1.27)
+				)
+				(hide yes)
+			)
+		)
+		(property "Description" "Resistor"
+			(at 93.98 78.74 0)
+			(effects
+				(font
+					(size 1.27 1.27)
+				)
+				(hide yes)
+			)
+		)
+		(pin "1"
+		)
+		(pin "2"
+		)
+		(instances
+			(project "main"
+				(path "/c11d1dbc-4db9-4712-8d1d-5f6f7086cded/e3db07b5-d47c-4d55-bf51-a423335924fb/520906bd-83a5-460c-87a5-c5c25b3f3979"
+					(reference "R148")
+					(unit 1)
+				)
+			)
 		)
 	)
@@
 					(unit 1)
 				)
+			)
+		)
+	)
+	(symbol
+		(lib_id "Device:R")
+		(at 93.98 163.83 0)
+		(mirror y)
+		(unit 1)
+		(exclude_from_sim no)
+		(in_bom yes)
+		(on_board yes)
+		(dnp yes)
+		(property "Reference" "R149"
+			(at 89.662 162.306 0)
+			(effects
+				(font
+					(size 1.27 1.27)
+				)
+			)
+		)
+		(property "Value" "10k"
+			(at 89.662 165.1 0)
+			(effects
+				(font
+					(size 1.27 1.27)
+				)
+			)
+		)
+		(property "Footprint" "Resistor_SMD:R_0805_2012Metric"
+			(at 95.758 163.83 90)
+			(effects
+				(font
+					(size 1.27 1.27)
+				)
+				(hide yes)
+			)
+		)
+		(property "Datasheet" "~"
+			(at 93.98 163.83 0)
+			(effects
+				(font
+					(size 1.27 1.27)
+				)
+				(hide yes)
+			)
+		)
+		(property "Description" "Resistor"
+			(at 93.98 163.83 0)
+			(effects
+				(font
+					(size 1.27 1.27)
+				)
+				(hide yes)
+			)
+		)
+		(pin "1"
+		)
+		(pin "2"
+		)
+		(instances
+			(project "main"
+				(path "/c11d1dbc-4db9-4712-8d1d-5f6f7086cded/e3db07b5-d47c-4d55-bf51-a423335924fb/520906bd-83a5-460c-87a5-c5c25b3f3979"
+					(reference "R149")
+					(unit 1)
+				)

Commit message: footprints set/changed
Parts:
- U25, U26: footprint (none) -> Package_SO:SOIC-20W_7.5x12.8mm_P1.27mm
Changed lines of the file:
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@@
 			)
 		)
-		(property "Footprint" ""
+		(property "Footprint" "Package_SO:SOIC-20W_7.5x12.8mm_P1.27mm"
 			(at 114.3 147.32 0)
 			(effects
@@
 			)
 		)
-		(property "Footprint" ""
+		(property "Footprint" "Package_SO:SOIC-20W_7.5x12.8mm_P1.27mm"
 			(at 114.3 62.23 0)
 			(effects
